File: A130XE_KB_MX/A130XE_KB_MX.kicad_pcb (KiCad board)
At the start: 2 copper layers, 330 x 131 mm, 76 parts, among them J1 34 pin RIBBON KEYBOARD CABLE, J2 Conn_01x02_Male, SW1 KS_RESET, SW10 K_5, SW11 K_I, SW12 K_T, SW13 K_G, SW14 K_SPACE, SW15 K_B, SW16 K_K, SW17 KS_SELECT, SW18 K_4, SW19 K_O, SW2 K_6, SW20 K_R, SW21 K_F, SW22 K_M, SW23 K_V, SW24 K_L, SW25 K_3, SW26 K_P, SW27 K_E, SW28 K_D, SW29 KS_START, SW3 K_U, SW30 K_comma, SW31 K_comdot, SW32 K_C, SW33 K_dot, SW34 K_2, SW35 K_minus, SW36 K_W, SW37 K_S, SW38 K_X, SW39 K_plus, SW4 K_Y, SW40 K_1, SW41 K_equal, SW42 K_Q, SW43 K_A, SW44 K_slash, SW45 K_asterisk, SW46 K_Z, SW47 K_ATARI, SW48 K_ESC, SW49 K_RETURN, SW5 K_H, SW50 K_TAB, SW51 K_CAPS, SW52 K_CTRL, SW53 K_LSHIFT, SW54 K_RSHIFT, SW55 K_BRK, SW56 K_DEL, SW57 K_GT, SW58 K_LT, SW59 K_0, SW6 K_N, SW60 K_9, SW61 K_8, SW62 K_7, SW63 K_SPACE_1, SW64 K_SPACE_2, SW65 K_F1, SW66 K_F2, SW67 K_F3, SW68 K_F4, SW7 KS_HELP, SW8 K_J, SW9 KS_OPTION

Commit message: Adapted for new positioning and removed error DRC on PCB
Parts:
- renumbered G*** to READY
Routing:
- net IN_2: track 297.0 -> 253.4 mm
- net IN_7: track 316.0 -> 274.1 mm, vias 5 -> 1
- net IN_5: track 326.2 -> 303.0 mm
- net START: track 148.8 -> 135.7 mm, vias 0 -> 1
- net RSC: track 402.2 -> 392.4 mm, vias 3 -> 1
- net IN_3: track 437.3 -> 427.6 mm, vias 1 -> 0
- net OPTION: track 143.1 -> 135.7 mm, vias 1 -> 0
- net GND: track 461.5 -> 468.3 mm, vias 1 -> 0
- net IN_4: track 349.5 -> 356.2 mm
- net OUT_4: track 281.6 -> 287.1 mm
- net OUT_0: track 305.8 -> 311.1 mm
- net IN_0: track 400.5 -> 396.2 mm, vias 1 -> 0
- net IN_1: track 325.1 -> 321.7 mm
- net OUT_1: track 221.7 -> 218.3 mm
- net OUT_6: track 221.4 -> 218.1 mm
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Other:
- net class +5V: trace_width 0.4 -> 0.35

Commit message: Regenerated after V2 (HELP, START, ..., RESET) are created from json file too. New plate & build web service with: http://www.keyboardcad.com
Parts:
- moved SW7 1.75 mm to (237.8, 89.9)
- moved SW29 1.34 mm to (266.3, 89.9)
- moved SW17 0.89 mm to (294.9, 89.9)
- moved SW9 0.55 mm to (323.5, 89.9)
- moved SW1 0.14 mm to (352.1, 89.9)
Routing:
- net IN_1: track 321.7 -> 336.5 mm
- net IN_3: track 427.6 -> 439.5 mm
- net OUT_5: track 482.8 -> 493.4 mm
- net IN_0: track 396.2 -> 389.8 mm
- net SELECT: track 150.8 -> 157.2 mm
- net OPTION: track 135.7 -> 130.6 mm
- net IN_4: track 356.2 -> 351.7 mm
- net OUT_1: track 218.3 -> 221.7 mm
- net RSC: track 392.4 -> 395.4 mm, vias 1 -> 0
- net GND: track 468.3 -> 465.8 mm
- net IN_5: track 303.0 -> 300.7 mm
- net IN_6: track 301.9 -> 302.9 mm
- net START: track 135.7 -> 135.0 mm
Other:
- board text added: "RSHIFT"
- board text added: "V2"

Commit message: F3 and F4 were inverted. Now they works fine. Thanks to OS ROM SELF-TEST Keyboard test.
Connections:
- SW67 pad 2: IN_3 -> IN_4
- SW68 pad 2: IN_4 -> IN_3
Routing:
- net RSC: track 395.4 -> 413.2 mm
- net IN_1: track 336.5 -> 322.3 mm
- net OUT_5: track 493.4 -> 484.5 mm
- net IN_4: track 351.7 -> 359.0 mm
- net SELECT: track 157.2 -> 150.5 mm
- net IN_3: track 439.5 -> 432.8 mm
- net IN_0: track 389.8 -> 395.9 mm
- net OUT_3: track 282.1 -> 276.6 mm
- net OPTION: track 130.6 -> 135.5 mm
- net OUT_2: track 277.2 -> 276.2 mm

Commit message: Updated with two jumpers for: 1- SHIFT ATARI (single shift) * DEFAULT 1-2 2- USB HID LSHIFT & RSHIFT 2-3
Parts:
- added J3: Conn_01x03_Male, Connector_PinHeader_2.54mm:PinHeader_1x03_P2.54mm_Vertical, F.Cu at (64.0, 185.0)
- added J4: Conn_01x03_Male, Connector_PinHeader_2.54mm:PinHeader_1x03_P2.54mm_Vertical, F.Cu at (262.0, 110.0)
- moved READY 3.48 mm to (57.0, 178.0)
Connections:
- J1 pad 25: Net-(J1-Pad25) -> LSC
- J1 pad 26: Net-(J1-Pad26) -> IN_FN
- SW1 pad 2: GND -> Net-(J4-Pad2)
- SW17 pad 2: GND -> Net-(J4-Pad2)
- SW29 pad 2: GND -> Net-(J4-Pad2)
- SW53 pad 2: RSC -> Net-(J3-Pad2)
- SW9 pad 2: GND -> Net-(J4-Pad2)
Routing:
- net LSC: track 0.00 -> 273.8 mm
- net IN_FN: track 0.00 -> 153.9 mm, vias 0 -> 1
- net Net-(J4-Pad2): track 0.00 -> 104.6 mm
- net GND: track 465.8 -> 362.0 mm
- net Net-(J3-Pad2): track 0.00 -> 24.0 mm
- net IN_1: track 322.3 -> 342.0 mm
- net OPTION: track 135.5 -> 116.6 mm
- net IN_4: track 359.0 -> 347.1 mm, vias 0 -> 1
- net IN_3: track 432.8 -> 422.1 mm, vias 0 -> 1
- net START: track 135.0 -> 145.3 mm, vias 1 -> 0
- net OUT_1: track 221.7 -> 231.5 mm
- net OUT_5: track 484.5 -> 494.0 mm
- net IN_6: track 302.9 -> 311.0 mm
- net RSC: track 413.2 -> 420.5 mm
- net OUT_0: track 311.0 -> 304.1 mm
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Other:
- board text added: "1-2 FN Keys tied to GND (ATARI) 2-3 FN Keys connected to IN_FN (USB HID)"
- board text added: "1-2 Single SHIFT (ATARI) 2-3 L/R SHIFT (USB HID)"

Commit message: Added some text into schematics. Renamed IN_FN as OUT_FN as it is an OUTPUT from microprocessor point of view.
Connections:
- net IN_FN renamed OUT_FN
Changed lines of the file:
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@@
   (net 33 "Net-(J2-Pad1)")
   (net 34 LSC)
-  (net 35 IN_FN)
-  (net 36 "Net-(J3-Pad2)")
-  (net 37 "Net-(J4-Pad2)")
+  (net 35 "Net-(J3-Pad2)")
+  (net 36 "Net-(J4-Pad2)")
+  (net 37 OUT_FN)
   (net_class Default "This is the default net class."
     (clearance 0.3)
@@
     (add_net IN_6)
     (add_net IN_7)
-    (add_net IN_FN)
     (add_net LSC)
     (add_net "Net-(D1-Pad2)")
@@
     (add_net OUT_6)
     (add_net OUT_7)
+    (add_net OUT_FN)
     (add_net RESET)
     (add_net RSC)
@@
     (pad "" np_thru_hole circle (at -2.54 5.08) (size 4 4) (drill 4) (layers *.Cu *.Mask))
     (pad 2 thru_hole circle (at -6.35 2.54) (size 2.2 2.2) (drill 1.5) (layers *.Cu *.Mask)
-      (net 37 "Net-(J4-Pad2)"))
+      (net 36 "Net-(J4-Pad2)"))
     (pad 1 thru_hole circle (at 0 0) (size 2.2 2.2) (drill 1.5) (layers *.Cu *.Mask)
       (net 23 OPTION))
@@
     (pad "" np_thru_hole circle (at -2.54 5.08) (size 4 4) (drill 4) (layers *.Cu *.Mask))
     (pad 2 thru_hole circle (at -6.35 2.54) (size 2.2 2.2) (drill 1.5) (layers *.Cu *.Mask)
-      (net 37 "Net-(J4-Pad2)"))
+      (net 36 "Net-(J4-Pad2)"))
     (pad 1 thru_hole circle (at 0 0) (size 2.2 2.2) (drill 1.5) (layers *.Cu *.Mask)
       (net 21 START))
@@
       (net 24 RESET))
     (pad 2 thru_hole circle (at -6.35 2.54) (size 2.2 2.2) (drill 1.5) (layers *.Cu *.Mask)
-      (net 37 "Net-(J4-Pad2)"))
+      (net 36 "Net-(J4-Pad2)"))
     (pad "" np_thru_hole circle (at -2.54 5.08) (size 4 4) (drill 4) (layers *.Cu *.Mask))
     (pad "" np_thru_hole circle (at -7.62 5.08) (size 1.7 1.7) (drill 1.7) (layers *.Cu *.Mask))
@@
       (net 22 SELECT))
     (pad 2 thru_hole circle (at -6.35 2.54) (size 2.2 2.2) (drill 1.5) (layers *.Cu *.Mask)
-      (net 37 "Net-(J4-Pad2)"))
+      (net 36 "Net-(J4-Pad2)"))
     (pad "" np_thru_hole circle (at -2.54 5.08) (size 4 4) (drill 4) (layers *.Cu *.Mask))
     (pad "" np_thru_hole circle (at -7.62 5.08) (size 1.7 1.7) (drill 1.7) (layers *.Cu *.Mask))
@@
       (net 6 OUT_5))
     (pad 2 thru_hole circle (at -6.35 2.54) (size 2.2 2.2) (drill 1.5) (layers *.Cu *.Mask)
-      (net 36 "Net-(J3-Pad2)"))
+      (net 35 "Net-(J3-Pad2)"))
     (pad "" np_thru_hole circle (at -2.54 5.08) (size 4 4) (drill 4) (layers *.Cu *.Mask))
     (pad "" np_thru_hole circle (at -7.62 5.08) (size 1.7 1.7) (drill 1.7) (layers *.Cu *.Mask))
@@
       (net 34 LSC))
     (pad 26 thru_hole oval (at 2.54 -30.48 270) (size 1.7 1.7) (drill 1) (layers *.Cu *.Mask)
-      (net 35 IN_FN))
+      (net 37 OUT_FN))
     (pad 27 thru_hole oval (at 0 -33.02 270) (size 1.7 1.7) (drill 1) (layers *.Cu *.Mask)
       (net 25 "Net-(J1-Pad27)"))
@@
       (net 20 RSC))
     (pad 2 thru_hole oval (at 0 2.54 180) (size 1.7 1.7) (drill 1) (layers *.Cu *.Mask)
-      (net 36 "Net-(J3-Pad2)"))
+      (net 35 "Net-(J3-Pad2)"))
     (pad 3 thru_hole oval (at 0 5.08 180) (size 1.7 1.7) (drill 1) (layers *.Cu *.Mask)
       (net 34 LSC))
@@
     (fp_line (start -0.635 -1.27) (end 1.27 -1.27) (layer F.Fab) (width 0.1))
     (pad 3 thru_hole oval (at 0 5.08 90) (size 1.7 1.7) (drill 1) (layers *.Cu *.Mask)
-      (net 35 IN_FN))
+      (net 37 OUT_FN))
     (pad 2 thru_hole oval (at 0 2.54 90) (size 1.7 1.7) (drill 1) (layers *.Cu *.Mask)
-      (net 37 "Net-(J4-Pad2)"))
+      (net 36 "Net-(J4-Pad2)"))
     (pad 1 thru_hole rect (at 0 0 90) (size 1.7 1.7) (drill 1) (layers *.Cu *.Mask)
       (net 1 GND))
@@
   (segment (start 117.6289 189.6385) (end 317.7185 189.6385) (width 0.3) (layer F.Cu) (net 34))
   (segment (start 317.7185 189.6385) (end 329.08 201) (width 0.3) (layer F.Cu) (net 34))
-  (segment (start 312.024 186.2815) (end 315.2107 186.2815) (width 0.3) (layer F.Cu) (net 35))
-  (segment (start 315.2107 186.2815) (end 326.7824 197.8532) (width 0.3) (layer F.Cu) (net 35))
-  (segment (start 326.7824 197.8532) (end 337.9354 197.8532) (width 0.3) (layer F.Cu) (net 35))
-  (segment (start 337.9354 197.8532) (end 340.555 200.4728) (width 0.3) (layer F.Cu) (net 35))
-  (segment (start 340.555 200.4728) (end 340.555 204.0688) (width 0.3) (layer F.Cu) (net 35))
-  (segment (start 340.555 204.0688) (end 339.7671 204.8567) (width 0.3) (layer F.Cu) (net 35))
-  (segment (start 339.7671 204.8567) (end 330.3967 204.8567) (width 0.3) (layer F.Cu) (net 35))
-  (segment (start 330.3967 204.8567) (end 329.08 203.54) (width 0.3) (layer F.Cu) (net 35))
-  (segment (start 267.08 110) (end 281.793 110) (width 0.3) (layer B.Cu) (net 35))
-  (segment (start 281.793 110) (end 302.8402 131.0472) (width 0.3) (layer B.Cu) (net 35))
-  (segment (start 302.8402 131.0472) (end 302.8402 143.3398) (width 0.3) (layer B.Cu) (net 35))
-  (segment (start 302.8402 143.3398) (end 312.024 152.5236) (width 0.3) (layer B.Cu) (net 35))
-  (segment (start 312.024 152.5236) (end 312.024 186.2815) (width 0.3) (layer B.Cu) (net 35))
-  (via (at 312.024 186.2815) (size 0.8) (layers F.Cu B.Cu) (net 35))
-  (segment (start 64 182.46) (end 86.73 182.46) (width 0.3) (layer F.Cu) (net 36))
-  (segment (start 86.73 182.46) (end 87.65 181.54) (width 0.3) (layer F.Cu) (net 36))
-  (segment (start 261.3423 92.46) (end 288.54 92.46) (width 0.3) (layer F.Cu) (net 37))
-  (segment (start 259.99 92.43) (end 260.02 92.46) (width 0.3) (layer F.Cu) (net 37))
-  (segment (start 260.02 92.46) (end 261.3423 92.46) (width 0.3) (layer F.Cu) (net 37))
-  (segment (start 264.54 108.6997) (end 261.3423 105.502) (width 0.3) (layer F.Cu) (net 37))
-  (segment (start 261.3423 105.502) (end 261.3423 92.46) (width 0.3) (layer F.Cu) (net 37))
-  (segment (start 264.54 110) (end 264.54 108.6997) (width 0.3) (layer F.Cu) (net 37))
-  (segment (start 288.54 92.46) (end 317.16 92.46) (width 0.3) (layer F.Cu) (net 37))
-  (segment (start 317.16 92.46) (end 317.19 92.43) (width 0.3) (layer F.Cu) (net 37))
-  (segment (start 345.74 92.43) (end 317.19 92.43) (width 0.3) (layer F.Cu) (net 37))
+  (segment (start 312.024 186.2815) (end 315.2107 186.2815) (width 0.3) (layer F.Cu) (net 37))
+  (segment (start 315.2107 186.2815) (end 326.7824 197.8532) (width 0.3) (layer F.Cu) (net 37))
+  (segment (start 326.7824 197.8532) (end 337.9354 197.8532) (width 0.3) (layer F.Cu) (net 37))
+  (segment (start 337.9354 197.8532) (end 340.555 200.4728) (width 0.3) (layer F.Cu) (net 37))
+  (segment (start 340.555 200.4728) (end 340.555 204.0688) (width 0.3) (layer F.Cu) (net 37))
+  (segment (start 340.555 204.0688) (end 339.7671 204.8567) (width 0.3) (layer F.Cu) (net 37))
+  (segment (start 339.7671 204.8567) (end 330.3967 204.8567) (width 0.3) (layer F.Cu) (net 37))
+  (segment (start 330.3967 204.8567) (end 329.08 203.54) (width 0.3) (layer F.Cu) (net 37))
+  (segment (start 267.08 110) (end 281.793 110) (width 0.3) (layer B.Cu) (net 37))
+  (segment (start 281.793 110) (end 302.8402 131.0472) (width 0.3) (layer B.Cu) (net 37))
+  (segment (start 302.8402 131.0472) (end 302.8402 143.3398) (width 0.3) (layer B.Cu) (net 37))
+  (segment (start 302.8402 143.3398) (end 312.024 152.5236) (width 0.3) (layer B.Cu) (net 37))
+  (segment (start 312.024 152.5236) (end 312.024 186.2815) (width 0.3) (layer B.Cu) (net 37))
+  (via (at 312.024 186.2815) (size 0.8) (layers F.Cu B.Cu) (net 37))
+  (segment (start 64 182.46) (end 86.73 182.46) (width 0.3) (layer F.Cu) (net 35))
+  (segment (start 86.73 182.46) (end 87.65 181.54) (width 0.3) (layer F.Cu) (net 35))
+  (segment (start 261.3423 92.46) (end 288.54 92.46) (width 0.3) (layer F.Cu) (net 36))
+  (segment (start 259.99 92.43) (end 260.02 92.46) (width 0.3) (layer F.Cu) (net 36))
+  (segment (start 260.02 92.46) (end 261.3423 92.46) (width 0.3) (layer F.Cu) (net 36))
+  (segment (start 264.54 108.6997) (end 261.3423 105.502) (width 0.3) (layer F.Cu) (net 36))
+  (segment (start 261.3423 105.502) (end 261.3423 92.46) (width 0.3) (layer F.Cu) (net 36))
+  (segment (start 264.54 110) (end 264.54 108.6997) (width 0.3) (layer F.Cu) (net 36))
+  (segment (start 288.54 92.46) (end 317.16 92.46) (width 0.3) (layer F.Cu) (net 36))
+  (segment (start 317.16 92.46) (end 317.19 92.43) (width 0.3) (layer F.Cu) (net 36))
+  (segment (start 345.74 92.43) (end 317.19 92.43) (width 0.3) (layer F.Cu) (net 36))
   (zone (net 1) (net_name GND) (layer F.Cu) (hatch edge 0.508)
     (connect_pads (clearance 0.508))

Commit message: New FPC cable. The Flat ribbon is for external USB HID Keyboard
Parts:
- added J5: 34 pin ribbon keyboard cable, Connector_IDC:IDC-Header_2x17_P2.54mm_Vertical, B.Cu at (368.0, 136.0)
- J1: value 34 pin RIBBON KEYBOARD CABLE -> Conn_01x32; footprint Connector_PinHeader_2.54mm:PinHeader_2x17_P2.54mm_Vertical -> RetroBitLab:FFC-1.25mm-RA-5204403245
- moved J1 32.5 mm to (331.0, 203.0), turned to 0 degrees
Connections:
- net Net-(D1-Pad2) renamed ~LED
Routing:
- net IN_2: track 253.6 -> 411.8 mm
- net IN_6: track 311.0 -> 468.0 mm
- net GND: track 362.0 -> 489.4 mm, vias 0 -> 1
- net ~LED: track 249.5 -> 374.6 mm, vias 0 -> 1
- net IN_7: track 275.4 -> 390.2 mm
- net +5V: track 0.00 -> 105.3 mm, vias 0 -> 1
- net IN_5: track 301.3 -> 404.6 mm
- net IN_1: track 342.0 -> 434.9 mm, vias 0 -> 1
- net OUT_4: track 292.3 -> 382.4 mm
- net IN_4: track 347.1 -> 430.6 mm, vias 1 -> 2
- net OUT_2: track 277.2 -> 355.8 mm, vias 1 -> 2
- net OUT_7: track 373.6 -> 445.7 mm
- net OUT_5: track 494.0 -> 564.7 mm, vias 1 -> 2
- net OUT_3: track 279.9 -> 349.7 mm
- net START: track 145.3 -> 215.0 mm, vias 0 -> 1
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Other:
- board size 330 x 131 mm -> 329 x 131 mm
- rule pad_to_mask_clearance: 0.051 -> 0
