File: A130XE_KB_MX/A130XE_KB_MX.kicad_pcb (KiCad board)
At the start: 2 copper layers, 329 x 131 mm, 79 parts, among them J1 Conn_01x32, J2 Conn_01x02_Male, J3 Conn_01x03_Male, J4 Conn_01x03_Male, J5 34 pin ribbon keyboard cable, SW1 KS_RESET, SW10 K_5, SW11 K_I, SW12 K_T, SW13 K_G, SW14 K_SPACE, SW15 K_B, SW16 K_K, SW17 KS_SELECT, SW18 K_4, SW19 K_O, SW2 K_6, SW20 K_R, SW21 K_F, SW22 K_M, SW23 K_V, SW24 K_L, SW25 K_3, SW26 K_P, SW27 K_E, SW28 K_D, SW29 KS_START, SW3 K_U, SW30 K_comma, SW31 K_comdot, SW32 K_C, SW33 K_dot, SW34 K_2, SW35 K_minus, SW36 K_W, SW37 K_S, SW38 K_X, SW39 K_plus, SW4 K_Y, SW40 K_1, SW41 K_equal, SW42 K_Q, SW43 K_A, SW44 K_slash, SW45 K_asterisk, SW46 K_Z, SW47 K_ATARI, SW48 K_ESC, SW49 K_RETURN, SW5 K_H, SW50 K_TAB, SW51 K_CAPS, SW52 K_CTRL, SW53 K_LSHIFT, SW54 K_RSHIFT, SW55 K_BRK, SW56 K_DEL, SW57 K_GT, SW58 K_LT, SW59 K_0, SW6 K_N, SW60 K_9, SW61 K_8, SW62 K_7, SW63 K_SPACE_1, SW64 K_SPACE_2, SW65 K_F1, SW66 K_F2, SW67 K_F3, SW68 K_F4, SW7 KS_HELP, SW8 K_J, SW9 KS_OPTION

Commit message: New layout. The spacebar is moved a little to the right, so the extra two keys are inverted to fit the computer plastic case hole.
Routing:
- net IN_6: track 468.0 -> 423.8 mm, vias 0 -> 1
- net IN_2: track 411.8 -> 378.7 mm
- net IN_4: track 430.6 -> 453.0 mm, vias 2 -> 1
- net RESET: track 165.3 -> 145.8 mm
- net OPTION: track 155.5 -> 174.4 mm
- net GND: track 489.4 -> 471.5 mm
- net RSC: track 437.8 -> 421.7 mm, vias 2 -> 1
- net OUT_0: track 331.9 -> 344.4 mm, vias 0 -> 1
- net OUT_1: track 272.3 -> 260.8 mm
- net OUT_5: track 564.7 -> 554.2 mm, vias 2 -> 1
- net +5V: track 105.3 -> 113.7 mm
- net OUT_6: track 236.4 -> 228.5 mm, vias 1 -> 2
- net IN_1: track 434.9 -> 427.6 mm
- net IN_0: track 437.5 -> 431.4 mm, vias 0 -> 1
- net IN_3: track 452.1 -> 458.2 mm, vias 2 -> 1
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Other:
- board text removed: "GPL3 License. OPENSOURCE PROJECT"

Commit message: Cleanup the extra unsused layers for Drawings.
Parts:
- moved SW63 147.6 mm to (289.1, 197.9)
- moved SW64 142.9 mm to (143.8, 197.9)
- moved SW14 4.80 mm to (217.7, 197.9)
Routing:
- net SELECT: track 172.7 -> 243.2 mm
- net IN_7: track 384.3 -> 426.4 mm
- net OUT_0: track 344.4 -> 319.3 mm, vias 1 -> 0
- net IN_4: track 453.0 -> 430.2 mm
- net OPTION: track 174.4 -> 153.8 mm, vias 1 -> 0
- net RSC: track 421.7 -> 437.1 mm, vias 1 -> 2
- net OUT_5: track 554.2 -> 569.2 mm, vias 1 -> 2
- net IN_3: track 458.2 -> 445.7 mm, vias 1 -> 2
- net GND: track 471.5 -> 459.8 mm
- net OUT_4: track 387.6 -> 376.7 mm, vias 0 -> 2
- net IN_1: track 427.6 -> 438.4 mm, vias 1 -> 0
- net OUT_3: track 350.8 -> 339.9 mm, vias 2 -> 3
- net LSC: track 338.1 -> 347.8 mm
- net IN_6: track 423.8 -> 433.3 mm
- net +5V: track 113.7 -> 121.8 mm
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
Commit message: New render for extra hole in the function keys (even if not needed really) and the spacebar 9U as alternative for modern spacebar 6.25U plus the other two keys
Parts:
- added G***: LOGO, RetroBitLab:atari_800_XL_BW_25x25, B.Cu at (181.0, 96.0)
- added GNUGPL: Symbol_GNU-GPL_CopperTop_Small, RetroBitLab:Symbol_GNU-GPL_SilkScreen_Small, B.Cu at (208.0, 95.0)
- added REF**: KiCad-Logo2_12mm_SilkScreen, Symbol:KiCad-Logo2_12mm_SilkScreen, F.Cu at (181.0, 92.0)
- added SW69: K_ATARI_SPACE_9U, RetroBitLab:SW_Cherry_MX1A_9u_PCB_3d, F.Cu at (217.7, 197.9)
- J1: footprint RetroBitLab:FFC-1.25mm-RA-5204403245 -> RetroBitLab:MOLEX-FFC-1.25mm-RA-52044-3245
- SW1, SW17, SW29, SW7, SW9: footprint RetroBitLab:SW_Cherry_MX1A_1.50u_PCB_3d -> RetroBitLab:SW_Cherry_MX1A_1.50u_ATARI_XE_PCB_3d
- moved READY 4.12 mm to (61.0, 177.0)
Routing:
- net SELECT: track 243.2 -> 183.1 mm, vias 1 -> 2
- net OPTION: track 153.8 -> 191.5 mm, vias 0 -> 2
- net OUT_7: track 442.2 -> 469.1 mm
- net OUT_6: track 230.3 -> 256.0 mm, vias 0 -> 1
- net OUT_4: track 376.7 -> 400.5 mm, vias 2 -> 1
- net LSC: track 347.8 -> 369.2 mm, vias 1 -> 2
- net IN_6: track 433.3 -> 452.9 mm
- net OUT_2: track 362.6 -> 380.9 mm
- net IN_2: track 382.0 -> 400.1 mm
- net +5V: track 121.8 -> 139.5 mm, vias 1 -> 2
- net OUT_1: track 260.9 -> 278.1 mm, vias 0 -> 1
- net START: track 211.6 -> 228.5 mm, vias 1 -> 2
- net IN_0: track 434.3 -> 449.3 mm, vias 2 -> 4
- net OUT_5: track 569.2 -> 583.7 mm, vias 2 -> 3
- net OUT_3: track 339.9 -> 352.9 mm, vias 3 -> 2
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Other:
- board text added: "9U SPACEBAR"
- board text added: "FFC Slim Cable"
- board text added: "GPL3 License. OPENSOURCE PROJECT"
- board text added: "https://github.com/gianlucarenzi/A130KB_MX"
