File: Atari130MX/Atari130MX.kicad_pcb (KiCad board)
At the start: 2 copper layers, 329.2 x 129.3 mm, 89 parts, among them J1 Conn_01x32, J2 Conn_01x26, J3 Conn_01x14, SW1 SW_Push_45deg, SW10 SW_Push_45deg, SW2 SW_Push_45deg, SW3 SW_Push_45deg, SW4 SW_Push_45deg, SW5 SW_Push_45deg, SW6 SW_Push_45deg, SW7 SW_Push_45deg, SW8 SW_Push_45deg, SW9 SW_Push_45deg, U1 PICO_RP2040

Commit message: BUG for LALT & RALT when used in Atari mode. Wrong ROW8 it must be ROW7 Tracks size increased, expecially for GND/POWER signals Added 9U spacebar and stabilizers like Atari keycaps. This is PCB only. The Plate is not compatible with it, at the moment...
Parts:
- added SW1: SPC 9U, RetroBit:SW_Cherry_MX1A_9u_PCB_3d, F.Cu at (189.4, 135.3)
- L7: renamed from L1; moved to B.Cu
- SW10: renamed from SWSpc2; value SW_Push_45deg -> Right-Alt
- SW11: renamed from SWJ1; value SW_Push_45deg -> J
- SW12: renamed from SWH1; value SW_Push_45deg -> H
- SW13: renamed from SWSpc3; value SW_Push_45deg -> SPC
- SW14: renamed from SWHlp1; value SW_Push_45deg -> Help
- SW15: renamed from SW3; value SW_Push_45deg -> 8
- SW16: renamed from SW4; value SW_Push_45deg -> 5
- SW17: renamed from SWI1; value SW_Push_45deg -> I
- SW18: renamed from SWT1; value SW_Push_45deg -> T
- SW19: renamed from SWK1; value SW_Push_45deg -> K
- SW2: renamed from SWSpc1; value SW_Push_45deg -> Left-Alt
- SW20: renamed from SWG1; value SW_Push_45deg -> G
- SW21: renamed from SWM1; value SW_Push_45deg -> M
- SW22: renamed from SWB1; value SW_Push_45deg -> B
- SW23: renamed from SW5; value SW_Push_45deg -> 9
- SW24: renamed from SW6; value SW_Push_45deg -> 4
- SW25: renamed from SWO1; value SW_Push_45deg -> O
- SW26: renamed from SWR1; value SW_Push_45deg -> R
- SW27: renamed from SWL1; value SW_Push_45deg -> L
- SW28: renamed from SWF1; value SW_Push_45deg -> F
- SW29: renamed from SWComma1; value SW_Push_45deg -> ,
- SW3: renamed from SW1; value SW_Push_45deg -> 7
- SW30: renamed from SWV1; value SW_Push_45deg -> V
- SW31: renamed from SW7; value SW_Push_45deg -> 0
- SW32: renamed from SW8; value SW_Push_45deg -> 3
- SW33: renamed from SWP1; value SW_Push_45deg -> P
- SW34: renamed from SWE1; value SW_Push_45deg -> E
- SW35: renamed from SWSemi1; value SW_Push_45deg -> ;
- SW36: renamed from SWD1; value SW_Push_45deg -> D
- SW37: renamed from SWPeriod1; value SW_Push_45deg -> .
- SW38: renamed from SWC1; value SW_Push_45deg -> C
- SW39: renamed from SWLT1; value SW_Push_45deg -> <
- SW4: renamed from SW2; value SW_Push_45deg -> 6
- SW40: renamed from SW9; value SW_Push_45deg -> 2
- SW41: renamed from SWDash1; value SW_Push_45deg -> -
- SW42: renamed from SWW1; value SW_Push_45deg -> W
- SW43: renamed from SWPlus1; value SW_Push_45deg -> +
- SW44: renamed from SWS1; value SW_Push_45deg -> S
- SW45: renamed from SWSlash1; value SW_Push_45deg -> /
- SW46: renamed from SWX1; value SW_Push_45deg -> X
- SW47: renamed from SWGT1; value SW_Push_45deg -> >
- SW48: renamed from SW10; value SW_Push_45deg -> 1
- SW49: renamed from SWEqual1; value SW_Push_45deg -> =
- SW5: renamed from SWU1; value SW_Push_45deg -> U
- SW50: renamed from SWQ1; value SW_Push_45deg -> Q
- SW51: renamed from SWStar1; value SW_Push_45deg -> *
- SW52: renamed from SWA1; value SW_Push_45deg -> A
- SW53: renamed from SWInv1; value SW_Push_45deg -> FUJI
- SW54: renamed from SWZ1; value SW_Push_45deg -> Z
- SW55: renamed from SWDel1; value SW_Push_45deg -> Del
- SW56: renamed from SWEsc1; value SW_Push_45deg -> Esc
- SW57: renamed from SWRet1; value SW_Push_45deg -> Return
- SW58: renamed from SWTab1; value SW_Push_45deg -> Tab
- SW59: renamed from SWFn3; value SW_Push_45deg -> F2
- SW6: renamed from SWY1; value SW_Push_45deg -> Y
- SW60: renamed from SWCps1; value SW_Push_45deg -> Caps
- SW61: renamed from SWFn4; value SW_Push_45deg -> F4
- SW62: renamed from SWBrk1; value SW_Push_45deg -> Break
- SW63: renamed from SWCtl1; value SW_Push_45deg -> Ctrl
- SW64: renamed from SWRightSft1; value SW_Push_45deg -> RSC
- SW65: renamed from SWLeftSft1; value SW_Push_45deg -> LSC
- SW66: renamed from SWStart1; value SW_Push_45deg -> Start
- SW67: renamed from SWSelect1; value SW_Push_45deg -> Select
- SW68: renamed from SWOption1; value SW_Push_45deg -> Option
- SW69: renamed from SWReset1; value SW_Push_45deg -> Reset
- SW7: renamed from SWFn1; value SW_Push_45deg -> F1
- SW8: renamed from SWN1; value SW_Push_45deg -> N
- SW9: renamed from SWFn2; value SW_Push_45deg -> F3
- moved L7 8.61 mm to (279.7, 49.1), turned to 180 degrees
- renumbered L2 to L1, L3 to L2, L4 to L3, L5 to L4, L6 to L5, L7 to L6
Connections:
- JP1 pad 3: ROW_8 -> ROW_7
- JP2 pad 3: ROW_8 -> ROW_7
Routing:
- net ROW_8: track 0.00 -> 590.9 mm
- net COL_2: track 0.00 -> 542.1 mm
- net COL_7: track 0.00 -> 511.1 mm, vias 0 -> 2
- net GND: track 0.00 -> 504.2 mm, vias 0 -> 4
- net ROW_7: track 0.00 -> 492.6 mm
- net ROW_5: track 0.00 -> 483.6 mm, vias 0 -> 1
- net COL_9: track 0.00 -> 459.9 mm, vias 0 -> 2
- net COL_6: track 0.00 -> 450.3 mm, vias 0 -> 1
- net COL_8: track 0.00 -> 443.8 mm, vias 0 -> 2
- net COL_5: track 0.00 -> 442.9 mm, vias 0 -> 1
- net COL_4: track 0.00 -> 439.3 mm, vias 0 -> 1
- net COL_1: track 0.00 -> 436.6 mm, vias 0 -> 1
- net COL_3: track 0.00 -> 430.1 mm, vias 0 -> 1
- net ROW_6: track 0.00 -> 428.0 mm, vias 0 -> 1
- net LED: track 0.00 -> 406.3 mm
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- added copper zone on B.Cu, net GND
- added copper zone on F.Cu, net GND
Other:
- net class Default: trace_width 0.25 -> 0.4
- net class GND added: clearance 0.2, trace_width 0.5, via_dia 0.8, via_drill 0.4
- net class POWER added: clearance 0.2, trace_width 0.45, via_dia 0.8, via_drill 0.4
- board text added: "JP3 2-3 ATARI SHIFT BOTH JP3 1-2 LSHIFT JP4 1-2 ATARI & Pi Pico GND Fn KEYS JP4 2-3 USB HID OUT_Fn"
- board text added: "Left Alt"
- board text added: "Right Alt"
- board text added: "spacebar 6.25u 9u"
- board text removed: "JP3 2-3 ATARI SHIFT BOTH JP3 1-2 LSHIFT JP4 1-2 ATARI GND Fn KEYS JP4 2-3 USB HID OUT_Fn"

Commit message: Added extra holes for 6.25U, 9U and stabilizers holes. Added extra holes for mounting on top cover if exist.
Parts:
- added H5: MountingHole, MountingHole:MountingHole_3.2mm_M3, F.Cu at (27.0, 138.0)
- added H6: MountingHole, MountingHole:MountingHole_3.2mm_M3, F.Cu at (27.0, 27.5)
- added H7: MountingHole, MountingHole:MountingHole_3.2mm_M3, F.Cu at (348.3, 27.5)
- added H8: MountingHole, MountingHole:MountingHole_3.2mm_M3, F.Cu at (348.3, 148.2)
- SW10: footprint Atari130MX:SW_Kailh_1.50u_PCB -> Atari130MX:SW_Kailh_1.25u_PCB
- SW2: footprint Atari130MX:SW_Kailh_1.25u_PCB -> Atari130MX:SW_Kailh_1.50u_PCB
- moved L2 4.55 mm to (46.8, 143.0)
- moved SW2 2.46 mm to (113.0, 140.4)
- moved SW10 2.40 mm to (258.3, 140.4)
Routing:
- net COL_1: track 436.6 -> 473.0 mm, vias 1 -> 2
- net ROW_5: track 483.6 -> 452.2 mm, vias 1 -> 2
- net POWER: track 404.4 -> 380.8 mm, vias 1 -> 3
- net OUT_FN: track 309.4 -> 331.9 mm
- net COL_8: track 443.8 -> 466.2 mm, vias 2 -> 1
- net ROW_6: track 428.0 -> 411.8 mm
- net ROW_7: track 492.6 -> 476.5 mm, vias 0 -> 1
- net ROW_8: track 590.9 -> 575.0 mm
- net SWDIO: track 40.6 -> 52.9 mm
- net COL_3: track 430.1 -> 441.0 mm, vias 1 -> 0
- net ROW_1: track 333.4 -> 341.1 mm
- net Net-(JP1-Pad2): track 103.3 -> 110.7 mm
- net SWCLK: track 54.0 -> 47.0 mm
- net GND: track 504.2 -> 511.1 mm, vias 4 -> 3
- net COL_9: track 459.9 -> 466.7 mm, vias 2 -> 1
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
Commit message: Using Atari spacebar (not fully 9U lenght). Other keys layout must be adapted a little bit.
Parts:
- SW1: footprint RetroBit:SW_Cherry_MX1A_9u_PCB_3d -> Atari130MX:SW_Kailh_Atari_Space
- moved SW1 5.72 mm to (186.9, 140.4)
- moved SW2 5.27 mm to (118.3, 140.4)
- moved SW13 4.80 mm to (194.2, 135.4)
- moved SW10 4.78 mm to (263.1, 140.4)
Routing:
- net Net-(JP2-Pad2): track 252.3 -> 262.1 mm
- net Net-(JP1-Pad2): track 110.7 -> 116.0 mm
Other:
- board text added: "(c) Bertrand Le Roy 2021 https://github.com/bleroy/3d-junkyard/tree/main/Atari130MX https://atariage.com/forums/profile/76850-screamingattheradio/ https://www.twitch.tv/screamingattheradio https://www.youtube.com/channel/UCyaCK4oVWf1ty618W-MJcrg Modified by Gianluca Renzi 2022-01"
- board text added: "130 MX Keyboard Rev. D"
- board text removed: "130 MX Keyboard Rev. E"

Commit message: It's simpler to use a (almost) standard 7U spacebar and two 1u extra keys. In that way, the holes needed are only for extra 9U stabilizers. Even the plate gets simpler.
Parts:
- removed the SW1 at (186.9, 140.4)
- removed the SW10 at (263.1, 140.4)
- removed the SW13 at (194.2, 135.4)
- removed the SW2 at (118.3, 140.4)
- added SW50: 9U SPC, RetroBit:SW_Cherry_MX1A_9u_PCB_noSwitch, F.Cu at (192.0, 135.3)
- added SW52: 7U SPC, RetroBit:MXOnly-7U-NoLED, F.Cu at (189.5, 140.4)
- added SW68: Left-Alt, Atari130MX:SW_Kailh_1.00u_PCB, F.Cu at (113.2, 140.3)
- added SW69: Right-Alt, Atari130MX:SW_Kailh_1.00u_PCB, F.Cu at (265.8, 140.4)
- renumbered J3 to J1, J1 to J3, JP4 to JP1, JP3 to JP2, JP1 to JP3, JP2 to JP4, L7 to L1, L1 to L2, L4 to L3, L2 to L4, L3 to L7, SW3 to SW1, SW67 to SW10, SW68 to SW11, SW69 to SW12, SW4 to SW13, SW16 to SW14, SW24 to SW15, SW32 to SW16, SW40 to SW17, SW48 to SW18, SW56 to SW19, SW15 to SW2, SW5 to SW20, SW17 to SW21, SW25 to SW22, SW33 to SW23, SW41 to SW24, SW49 to SW25, SW57 to SW26, SW6 to SW27, SW18 to SW28, SW26 to SW29, SW23 to SW3, SW34 to SW30, SW42 to SW31, SW50 to SW32, SW58 to SW33, SW7 to SW34, SW11 to SW35, SW19 to SW36, SW27 to SW37, SW35 to SW38, SW43 to SW39, SW31 to SW4, SW51 to SW40, SW59 to SW41, SW63 to SW42, SW12 to SW43, SW20 to SW44, SW28 to SW45, SW36 to SW46, SW44 to SW47, SW52 to SW48, SW60 to SW49, SW39 to SW5, SW8 to SW51, SW21 to SW53, SW29 to SW54, SW37 to SW55, SW45 to SW56, SW53 to SW57, SW9 to SW58, SW14 to SW59, SW47 to SW6, SW22 to SW60, SW30 to SW61, SW38 to SW62, SW46 to SW63, SW54 to SW64, SW61 to SW65, SW64 to SW66, SW65 to SW67, SW55 to SW7, SW62 to SW8, SW66 to SW9
Routing:
- net ROW_6: track 411.8 -> 452.7 mm, vias 1 -> 0
- net ROW_4: track 400.6 -> 373.1 mm, vias 0 -> 1
- net COL_1: track 473.0 -> 445.5 mm, vias 2 -> 1
- net COL_9: track 466.7 -> 488.2 mm, vias 1 -> 2
- net OUT_FN: track 331.9 -> 311.5 mm
- net SWDIO: track 52.9 -> 34.4 mm
- net COL_8: track 466.2 -> 448.0 mm
- net GND: track 511.1 -> 527.3 mm, vias 3 -> 2
- net ROW_1: track 341.1 -> 356.9 mm, vias 2 -> 1
- net COL_3: track 441.0 -> 428.4 mm
- net Net-(JP3-Pad2): track 116.0 -> 106.9 mm
- net /LED-GP2: track 53.0 -> 45.7 mm, vias 0 -> 1
- net SWCLK: track 47.0 -> 41.6 mm
- net Net-(JP1-Pad2): track 341.5 -> 336.3 mm, vias 0 -> 1
- net ROW_2: track 340.4 -> 336.2 mm
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Other:
- board text added: "spacebar 7u 9u"
- board text removed: "spacebar 6.25u 9u"

Commit message: Removed the original FFC connector. This will lose any compatibility between two projects
Parts:
- removed the J2 at (323.0, 47.1)
- moved L1 56.5 mm to (336.2, 52.6)
- moved J2 47.9 mm to (301.2, 51.6), turned to 0 degrees
- moved L3 35.0 mm to (254.2, 46.6)
- moved JP1 20.2 mm to (28.2, 76.6)
- moved JP3 11.0 mm to (28.2, 86.6)
- moved JP4 9.85 mm to (28.2, 91.6)
- moved JP2 9.67 mm to (28.2, 81.6)
- moved D1 4.43 mm to (25.2, 144.6)
- renumbered J3 to J2
Routing:
- net GND: track 527.3 -> 431.6 mm, vias 2 -> 1
- net COL_7: track 511.7 -> 424.8 mm, vias 1 -> 2
- net ROW_6: track 452.7 -> 375.3 mm, vias 0 -> 1
- net COL_6: track 448.7 -> 373.0 mm, vias 0 -> 1
- net COL_4: track 437.8 -> 362.3 mm
- net COL_3: track 428.4 -> 355.4 mm, vias 0 -> 1
- net POWER: track 381.4 -> 309.3 mm
- net ROW_5: track 453.6 -> 383.6 mm
- net LED: track 409.8 -> 341.3 mm
- net COL_5: track 439.6 -> 371.1 mm
- net START: track 338.1 -> 277.2 mm, vias 1 -> 0
- net COL_1: track 445.5 -> 386.4 mm, vias 1 -> 0
- net COL_2: track 544.0 -> 486.9 mm
- net ROW_2: track 336.2 -> 279.9 mm, vias 1 -> 0
- net SELECT: track 328.3 -> 274.6 mm, vias 1 -> 0
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Other:
- board text added: "(c) Bertrand Le Roy 2021 https://github.com/bleroy/3d-junkyard/tree/main/Atari130MX https://atariage.com/forums/profile/76850-screamingattheradio/ https://www.twitch.tv/screamingattheradio https://www.youtube.com/channel/UCyaCK4oVWf1ty618W-MJcrg Modified by Gianluca Renzi Jan 2022"
- board text added: "130 MX Keyboard Rev. Jan 2022"
- board text added: "130MX Keyboard Rev. Jan 2022"
- board text added: "JP1 1-2 ATARI & Pi Pico GND Fn KEYS JP1 2-3 USB HID OUT_Fn JP2 2-3 ATARI SHIFT BOTH JP2 1-2 LEFT SHIFT"
- board text added: "JP3 1-2 LEFT ALT JP3 2-3 ATARI SPC JP4 1-2 RIGHT ALT JP4 2-3 ATARI SPC"
- board text removed: "(c) Bertrand Le Roy 2021 https://github.com/bleroy/3d-junkyard/tree/main/Atari130MX https://atariage.com/forums/profile/76850-screamingattheradio/ https://www.twitch.tv/screamingattheradio https://www.youtube.com/channel/UCyaCK4oVWf1ty618W-MJcrg Modified by Gianluca Renzi 2021-12"
- board text removed: "(c) Bertrand Le Roy 2021 https://github.com/bleroy/3d-junkyard/tree/main/Atari130MX https://atariage.com/forums/profile/76850-screamingattheradio/ https://www.twitch.tv/screamingattheradio https://www.youtube.com/channel/UCyaCK4oVWf1ty618W-MJcrg Modified by Gianluca Renzi 2022-01"
- board text removed: "130 MX Keyboard Rev. D"
- board text removed: "130MX Keyboard Rev. E"
- board text removed: "JP1 1-2 LALT JP1 2-3 ATARI SPC JP2 1-2 RALT JP2 2-3 ATARI SPC"
- board text removed: "JP3 2-3 ATARI SHIFT BOTH JP3 1-2 LSHIFT JP4 1-2 ATARI & Pi Pico GND Fn KEYS JP4 2-3 USB HID OUT_Fn"

Commit message: Updated to reflect the correct path for importing the PCB in FreeCad with the KicadStepUp plugin
Parts:
- U1: footprint Atari130MX:RPi_Pico_SMD_TH -> RetroBit:RPi_Pico_SMD_TH
