File: Atari130MX/Atari130MX.kicad_pcb (KiCad board)
At the start: 2 copper layers, 329.2 x 129.3 mm, 93 parts, among them J1 Conn_01x14, J2 Conn_01x32, SW1 7, SW10 Select, SW11 Option, SW12 Reset, SW13 6, SW14 5, SW15 4, SW16 3, SW17 2, SW18 1, SW19 Esc, SW2 8, SW20 U, SW21 I, SW22 O, SW23 P, SW24 -, SW25 =, SW26 Return, SW27 Y, SW28 T, SW29 R, SW3 9, SW30 E, SW31 W, SW32 Q, SW33 Tab, SW34 F1, SW35 J, SW36 K, SW37 L, SW38 ;, SW39 +, SW4 0, SW40 *, SW41 F2, SW42 Ctrl, SW43 H, SW44 G, SW45 F, SW46 D, SW47 S, SW48 A, SW49 Caps, SW5 <, SW50 9U SPC, SW51 N, SW52 7U SPC, SW53 M, SW54 ,, SW55 ., SW56 /, SW57 FUJI, SW58 F3, SW59 Help, SW6 >, SW60 B, SW61 V, SW62 C, SW63 X, SW64 Z, SW65 F4, SW66 RSC, SW67 LSC, SW68 Left-Alt, SW69 Right-Alt, SW7 Del, SW8 Break, SW9 Start, U1 PICO_RP2040

Commit message: Changed from switches with 3D CherryMX Switch, to switches with only the keycaps. They are much lighter for renderings The PCB should not be affected, but I redo a Plot just for sure.
Parts:
- SW1, SW13, SW14, SW15, SW16, SW17, SW18, SW19, SW2, SW20, SW21, SW22, SW23, SW24, SW25, SW27, SW28, SW29, SW3, SW30, SW31, SW32, SW35, SW36, SW37, SW38, SW39, SW4, SW40, SW43, SW44, SW45, SW46, SW47, SW48, SW5, SW51, SW53, SW54, SW55, SW56, SW57, SW6, SW60, SW61, SW62, SW63, SW64, SW68, SW69, SW7, SW8: footprint Atari130MX:SW_Kailh_1.00u_PCB -> Atari130MX:SW_Kailh_1.00u_PCB_noSwitch
- SW10, SW11, SW12, SW34, SW41, SW58, SW59, SW65, SW9: footprint Atari130MX:SW_Kailh_1.50u_Atari_Fn_PCB -> Atari130MX:SW_Kailh_1.50u_Atari_Fn_PCB_noSwitch
- SW26, SW33: footprint Atari130MX:SW_Kailh_1.50u_PCB -> Atari130MX:SW_Kailh_1.50u_PCB_noSwitch
- SW42, SW66: footprint Atari130MX:SW_Kailh_1.75u_PCB -> Atari130MX:SW_Kailh_1.75u_PCB_noSwitch
- SW49: footprint Atari130MX:SW_Kailh_1.25u_PCB -> Atari130MX:SW_Kailh_1.25u_PCB_noSwitch
- SW67: footprint Atari130MX:SW_Kailh_2.25u_PCB -> Atari130MX:SW_Kailh_2.25u_PCB_noSwitch
