File: A130XE_KB_MX/STM32F4XX_Hat/STM32F4XX_Hat.sch (KiCad schematic (older format))
At the start: 23 parts, among them J1 Conn_02x16_Odd_Even, J2 Conn_02x24_Odd_Even, J3 Conn_02x24_Odd_Even, J4 Conn_02x17_Counter_Clockwise, J5 Conn_01x32, J6 Conn_01x03

Commit message: RetroBitLab library
Parts:
- LOGO1: symbol AmigaComponents:LOGO -> RetroBitLab:LOGO
Changed lines of the file:
@@
 NoConn ~ 3700 1550
 $Comp
-L AmigaComponents:LOGO LOGO1
+L RetroBitLab:LOGO LOGO1
 U 1 1 61A9B360
 P 7350 5450
